File: self_balancing_bot_pcb/self_balancing_bot.kicad_pcb (KiCad board)
At the start: 2 copper layers, 6 parts, among them J1 Conn_01x08_Female, J2 Conn_01x06_Female, J3 Conn_01x04_Female, J4 Conn_01x06_Female, J5 Conn_01x02_Female

Commit message: autosave wala add
Parts:
- moved J4 218.2 mm to (124.2, 61.0)
- moved J2 211.0 mm to (124.2, 43.9)
- moved J3 187.3 mm to (98.3, 74.2), turned to -90 degrees
- moved J5 114.4 mm to (83.3, 74.2), turned to 90 degrees
- moved J1 79.0 mm to (98.0, 51.3)
- moved A1 45.6 mm to (109.5, 57.1)
Changed lines of the file:
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@@
   (net 34 "AD0")
   (footprint "Connector_PinHeader_2.54mm:PinHeader_1x02_P2.54mm_Vertical" (layer "F.Cu")
-    (at -30.558 85.09)
+    (at 83.307 74.168 90)
     (descr "Through hole straight pin header, 1x02, 2.54mm pitch, single row")
     (tags "Through hole pin header THT 1x02 2.54mm single row")
@@
     (property "Sheetname" "")
     (attr through_hole)
-    (fp_text reference "J5" (at 0 -2.33) (layer "F.SilkS")
-      (effects (font (size 1 1) (thickness 0.15)))
-    )
-    (fp_text value "Conn_01x02_Female" (at 0 4.87) (layer "F.Fab")
-      (effects (font (size 1 1) (thickness 0.15)))
-    )
-    (fp_text user "${REFERENCE}" (at 0 1.27 90) (layer "F.Fab")
+    (fp_text reference "J5" (at 0 -2.33 90) (layer "F.SilkS") hide
+      (effects (font (size 1 1) (thickness 0.15)))
+    )
+    (fp_text value "Conn_01x02_Female" (at 0 4.87 90) (layer "F.Fab") hide
+      (effects (font (size 1 1) (thickness 0.15)))
+    )
+    (fp_text user "${REFERENCE}" (at 0 1.27) (layer "F.Fab")
       (effects (font (size 1 1) (thickness 0.15)))
     )
@@
     (fp_line (start 1.27 -1.27) (end 1.27 3.81) (layer "F.Fab") (width 0.1))
     (fp_line (start 1.27 3.81) (end -1.27 3.81) (layer "F.Fab") (width 0.1))
-    (pad "1" thru_hole rect (at 0 0) (size 1.7 1.7) (drill 1) (layers *.Cu *.Mask)
+    (pad "1" thru_hole rect (at 0 0 90) (size 1.7 1.7) (drill 1) (layers *.Cu *.Mask)
       (net 18 "GND") (pinfunction "Pin_1") (pintype "passive"))
-    (pad "2" thru_hole oval (at 0 2.54) (size 1.7 1.7) (drill 1) (layers *.Cu *.Mask)
+    (pad "2" thru_hole oval (at 0 2.54 90) (size 1.7 1.7) (drill 1) (layers *.Cu *.Mask)
       (net 15 "VCC") (pinfunction "Pin_2") (pintype "passive"))
     (model "${KICAD6_3DMODEL_DIR}/Connector_PinHeader_2.54mm.3dshapes/PinHeader_1x02_P2.54mm_Vertical.wrl"
@@
   )
   (footprint "Connector_PinHeader_2.54mm:PinHeader_1x06_P2.54mm_Vertical" (layer "F.Cu")
-    (at -85.266 18.796)
+    (at 124.206 43.942)
     (descr "Through hole straight pin header, 1x06, 2.54mm pitch, single row")
     (tags "Through hole pin header THT 1x06 2.54mm single row")
@@
     (property "Sheetname" "")
     (attr through_hole)
-    (fp_text reference "J2" (at 0 -2.33) (layer "F.SilkS")
-      (effects (font (size 1 1) (thickness 0.15)))
-    )
-    (fp_text value "Conn_01x06_Female" (at 0 15.03) (layer "F.Fab")
+    (fp_text reference "J2" (at 0 -2.33) (layer "F.SilkS") hide
+      (effects (font (size 1 1) (thickness 0.15)))
+    )
+    (fp_text value "Conn_01x06_Female" (at 0 15.03) (layer "F.Fab") hide
       (effects (font (size 1 1) (thickness 0.15)))
     )
@@
   )
   (footprint "Connector_PinHeader_2.54mm:PinHeader_1x06_P2.54mm_Vertical" (layer "F.Cu")
-    (at -89.916 18.796)
+    (at 124.206 60.96)
     (descr "Through hole straight pin header, 1x06, 2.54mm pitch, single row")
     (tags "Through hole pin header THT 1x06 2.54mm single row")
@@
     (property "Sheetname" "")
     (attr through_hole)
-    (fp_text reference "J4" (at 0 -2.33) (layer "F.SilkS")
-      (effects (font (size 1 1) (thickness 0.15)))
-    )
-    (fp_text value "Conn_01x06_Female" (at 0 15.03) (layer "F.Fab")
+    (fp_text reference "J4" (at 0 -2.33) (layer "F.SilkS") hide
+      (effects (font (size 1 1) (thickness 0.15)))
+    )
+    (fp_text value "Conn_01x06_Female" (at 0 15.03) (layer "F.Fab") hide
       (effects (font (size 1 1) (thickness 0.15)))
     )
@@
   )
   (footprint "Connector_PinHeader_2.54mm:PinHeader_1x04_P2.54mm_Vertical" (layer "F.Cu")
-    (at -80.616 18.796)
+    (at 98.298 74.168 -90)
     (descr "Through hole straight pin header, 1x04, 2.54mm pitch, single row")
     (tags "Through hole pin header THT 1x04 2.54mm single row")
@@
     (property "Sheetname" "")
     (attr through_hole)
-    (fp_text reference "J3" (at 0 -2.33) (layer "F.SilkS")
-      (effects (font (size 1 1) (thickness 0.15)))
-    )
-    (fp_text value "Conn_01x04_Female" (at 0 9.95) (layer "F.Fab")
-      (effects (font (size 1 1) (thickness 0.15)))
-    )
-    (fp_text user "${REFERENCE}" (at 0 3.81 90) (layer "F.Fab")
+    (fp_text reference "J3" (at 0 -2.33 90) (layer "F.SilkS") hide
+      (effects (font (size 1 1) (thickness 0.15)))
+    )
+    (fp_text value "Conn_01x04_Female" (at 0 9.95 90) (layer "F.Fab") hide
+      (effects (font (size 1 1) (thickness 0.15)))
+    )
+    (fp_text user "${REFERENCE}" (at 0 3.81) (layer "F.Fab")
       (effects (font (size 1 1) (thickness 0.15)))
     )
@@
     (fp_line (start -1.27 8.89) (end -1.27 -0.635) (layer "F.Fab") (width 0.1))
     (fp_line (start -0.635 -1.27) (end 1.27 -1.27) (layer "F.Fab") (width 0.1))
-    (pad "1" thru_hole rect (at 0 0) (size 1.7 1.7) (drill 1) (layers *.Cu *.Mask)
+    (pad "1" thru_hole rect (at 0 0 270) (size 1.7 1.7) (drill 1) (layers *.Cu *.Mask)
       (net 15 "VCC") (pinfunction "Pin_1") (pintype "passive"))
-    (pad "2" thru_hole oval (at 0 2.54) (size 1.7 1.7) (drill 1) (layers *.Cu *.Mask)
+    (pad "2" thru_hole oval (at 0 2.54 270) (size 1.7 1.7) (drill 1) (layers *.Cu *.Mask)
       (net 18 "GND") (pinfunction "Pin_2") (pintype "passive"))
-    (pad "3" thru_hole oval (at 0 5.08) (size 1.7 1.7) (drill 1) (layers *.Cu *.Mask)
+    (pad "3" thru_hole oval (at 0 5.08 270) (size 1.7 1.7) (drill 1) (layers *.Cu *.Mask)
       (net 21 "RXD") (pinfunction "Pin_3") (pintype "passive"))
-    (pad "4" thru_hole oval (at 0 7.62) (size 1.7 1.7) (drill 1) (layers *.Cu *.Mask)
+    (pad "4" thru_hole oval (at 0 7.62 270) (size 1.7 1.7) (drill 1) (layers *.Cu *.Mask)
       (net 20 "TXD") (pinfunction "Pin_4") (pintype "passive"))
     (model "${KICAD6_3DMODEL_DIR}/Connector_PinHeader_2.54mm.3dshapes/PinHeader_1x04_P2.54mm_Vertical.wrl"
@@
   )
   (footprint "Library:Arduino Pro Mini" (layer "F.Cu")
-    (at 153.044 70.506)
-    (property "Sheetfile" "self_balancing_bot.kicad_sch")
-    (property "Sheetname" "")
-    (attr through_hole)
-    (fp_text reference "A1" (at 0.99 -16.06 unlocked) (layer "F.SilkS")
-      (effects (font (size 1 1) (thickness 0.15)))
-    )
-    (fp_text value "Arduino_Leonardo" (at 0.64 1.88 90 unlocked) (layer "F.Fab")
+    (at 109.474 57.15)
+    (property "Sheetfile" "self_balancing_bot.kicad_sch")
+    (property "Sheetname" "")
+    (attr through_hole)
+    (fp_text reference "A1" (at 0.99 -16.06 unlocked) (layer "F.SilkS") hide
+      (effects (font (size 1 1) (thickness 0.15)))
+    )
+    (fp_text value "Arduino_Leonardo" (at 0.64 1.88 90 unlocked) (layer "F.Fab") hide
       (effects (font (size 1 1) (thickness 0.15)))
     )
@@
   )
   (footprint "Connector_PinHeader_2.54mm:PinHeader_1x08_P2.54mm_Vertical" (layer "F.Cu")
-    (at 176.784 57.15)
+    (at 98.044 51.308)
     (descr "Through hole straight pin header, 1x08, 2.54mm pitch, single row")
     (tags "Through hole pin header THT 1x08 2.54mm single row")
@@
     (property "Sheetname" "")
     (attr through_hole)
-    (fp_text reference "J1" (at 0 -2.33) (layer "F.SilkS")
-      (effects (font (size 1 1) (thickness 0.15)))
-    )
-    (fp_text value "Conn_01x08_Female" (at 0 20.11) (layer "F.Fab")
-      (effects (font (size 1 1) (thickness 0.15)))
+    (fp_text reference "J1" (at 0 -2.33) (layer "F.SilkS") hide
+      (effects (font (size 1 1) (thickness 0.15)))
+    )
+    (fp_text value "Conn_01x08_Female" (at 0 20.11) (layer "F.Fab") hide
+      (effects (font (size 1 1) (thickness 0.15)) (justify mirror))
     )
     (fp_text user "${REFERENCE}" (at 0 8.89 90) (layer "F.Fab")
@@
     )
   )
-  (gr_rect (start 79.686 41.402) (end 229.686 111.402) (layer "F.SilkS") (width 0.4) (fill none))
+  (gr_rect (start 79.686 41.402) (end 141.986 86.868) (layer "F.SilkS") (width 0.4) (fill none))
 )
